Commit message: Task 1: replace 2D LiDAR with 16-ring 3D LiDAR
- VLP-16-class gpu_lidar: 16 rings (-15..+15 deg), 900 pts/ring, 0.4-100 m,
  10 Hz, 3 cm noise, on a 0.25 m mast (optical centre 0.67 m, no self-hits)
- bridge /lidar/points -> /points (sensor_msgs/PointCloud2)
- cloud_to_scan.py derives /scan from the cloud for slam_toolbox / Nav2
- sensor_test: +5 checks (layout, self-hits, ground height, canopy, rates);
  18/18 pass; motion 20/20 and orchard 11/11 re-verified
- RViz shows the point cloud; README updated (orchard visually checked by user)

Co-Authored-By: Claude Opus 5.5 <noreply@anthropic.com>

File: src/agri_ugv_description/urdf/agri_ugv.sensors.xacro (robot description, xacro)
@@ -7,5 +7,6 @@
   Frames:  imu_link, gps_link, lidar_link, camera_link (x forward),
            camera_optical_frame (z forward, x right: ROS optical convention).
-  Topics:  /imu, /gps/fix, /scan, /camera/image_raw, /camera/camera_info
+  Topics:  /imu, /gps/fix, /points (3D LiDAR), /scan (derived 2D),
+           /camera/image_raw, /camera/camera_info
 -->
 <robot xmlns:xacro="http://www.ros.org/wiki/xacro">
@@ -80,10 +81,17 @@
     </sensor>
   </gazebo>
-  <!-- ===================== 2D LiDAR on a short mast ===================== -->
+  <!-- ===================== 3D LiDAR (VLP-16 class) on a mast ===================== -->
+  <!-- 16 rings from -15 to +15 deg (2 deg apart), 900 points per ring (0.4 deg),
+       10 Hz, 0.4-100 m, +-3 cm noise: Velodyne VLP-16 datasheet values.
+       Gazebo topics: /lidar (multi-ring scan, not bridged) and /lidar/points
+       (bridged to ROS /points, sensor_msgs/PointCloud2).
+       A 2D /scan is derived from the near-horizontal points by cloud_to_scan.py. -->
+  <xacro:property name="lidar_mast_len" value="0.25"/>
+  <xacro:property name="lidar_body_h"   value="0.072"/>
   <xacro:if value="$(arg enable_lidar)">
     <link name="lidar_mast">
       <visual>
-        <origin xyz="0 0 0.05"/>
-        <geometry><cylinder radius="0.02" length="0.10"/></geometry>
+        <origin xyz="0 0 ${lidar_mast_len/2}"/>
+        <geometry><cylinder radius="0.02" length="${lidar_mast_len}"/></geometry>
         <material name="dark_grey"/>
       </visual>
@@ -96,13 +104,14 @@
     <link name="lidar_link">
       <visual>
-        <geometry><cylinder radius="0.04" length="0.07"/></geometry>
-        <material name="tyre_black"/>
+        <geometry><cylinder radius="0.0515" length="${lidar_body_h}"/></geometry>
+        <material name="hub_grey"/>
       </visual>
     </link>
-    <!-- scan plane ~0.52 m above ground: sees trunks, passes under the canopy -->
+    <!-- optical centre ~0.67 m above ground. High enough that the -15 deg ring
+         clears the top plate, GPS puck and camera (no self-hits). -->
     <joint name="lidar_joint" type="fixed">
       <parent link="lidar_mast"/>
       <child link="lidar_link"/>
-      <origin xyz="0 0 0.135"/>
+      <origin xyz="0 0 ${lidar_mast_len + lidar_body_h/2}"/>
     </joint>
     <gazebo reference="lidar_link">
@@ -110,5 +119,5 @@
         <always_on>true</always_on>
         <update_rate>10</update_rate>
-        <topic>scan</topic>
+        <topic>lidar</topic>
         <gz_frame_id>lidar_link</gz_frame_id>
         <visualize>false</visualize>
@@ -116,22 +125,22 @@
           <scan>
             <horizontal>
-              <samples>720</samples>
+              <samples>900</samples>
               <resolution>1</resolution>
               <min_angle>${-pi}</min_angle>
-              <max_angle>${pi - 2*pi/720}</max_angle>
+              <max_angle>${pi - 2*pi/900}</max_angle>
             </horizontal>
             <vertical>
-              <samples>1</samples>
+              <samples>16</samples>
               <resolution>1</resolution>
-              <min_angle>0</min_angle>
-              <max_angle>0</max_angle>
+              <min_angle>${radians(-15)}</min_angle>
+              <max_angle>${radians(15)}</max_angle>
             </vertical>
           </scan>
           <range>
-            <min>0.20</min>
-            <max>20.0</max>
+            <min>0.40</min>
+            <max>100.0</max>
             <resolution>0.01</resolution>
           </range>
-          <noise><type>gaussian</type><mean>0.0</mean><stddev>0.01</stddev></noise>
+          <noise><type>gaussian</type><mean>0.0</mean><stddev>0.03</stddev></noise>
         </lidar>
       </sensor>

Commit message: Task 3: RTK GPS with a base station on a known point
- models/rtk_base_station: tripod, antenna and radio, GNSS receiver (rtk_base/navsat)
  placed in both worlds (orchard via generate_orchard.py, same seed: only additions)
- rtk_gnss.py: common satellite/atmosphere error, base-station corrections at 1 Hz,
  /gps/raw (standalone ~1.5 m) and /gps/fix (RTK ~2 cm, status GBAS_FIX,
  fallback to standalone when rtk_enabled is false or corrections are stale)
- robot receiver: 1 cm noise on /gps/navsat
- rtk_test.py (11 checks) added to run_tests.sh

Tests: rtk 11/11, motion 20/20, orchard 11/11, sensor 22/22.

Co-Authored-By: Claude Opus 5.5 <noreply@anthropic.com>

File: src/agri_ugv_description/urdf/agri_ugv.sensors.xacro (robot description, xacro)
@@ -7,5 +7,5 @@
   Frames:  imu_link, gps_link, lidar_link, camera_link (x forward),
            camera_optical_frame (z forward, x right: ROS optical convention).
-  Topics:  /imu, /gps/fix, /points (3D LiDAR), /scan (derived 2D),
+  Topics:  /imu, /gps/navsat (-> rtk_gnss.py -> /gps/fix), /points (3D LiDAR), /scan (derived 2D),
            /camera/image_raw, /camera/depth/image_raw, /camera/camera_info
 -->
@@ -52,5 +52,8 @@
   </gazebo>
   <!-- ===================== GPS (NavSat) ===================== -->
-  <xacro:property name="gps_noise_m" value="0.3"/>  <!-- horizontal 1-sigma, metres -->
+  <!-- RTK GNSS receiver. Gazebo gives the true antenna position + receiver noise;
+       rtk_gnss.py adds the satellite/atmosphere error and the base-station
+       corrections, and publishes /gps/raw (standalone) and /gps/fix (RTK). -->
+  <xacro:property name="gps_noise_m" value="0.01"/>  <!-- receiver noise, horizontal 1-sigma, metres -->
   <link name="gps_link">
     <visual>
@@ -68,13 +71,12 @@
       <always_on>true</always_on>
       <update_rate>10</update_rate>
-      <topic>gps/fix</topic>
+      <topic>gps/navsat</topic>
       <gz_frame_id>gps_link</gz_frame_id>
       <navsat>
         <!-- Gazebo applies horizontal noise to latitude/longitude in DEGREES:
-             ${gps_noise_m} m / 111320 m-per-degree. 0.3 m = SBAS-class receiver;
-             use ~0.02 m for RTK. Vertical noise is in metres. -->
+             ${gps_noise_m} m / 111320 m-per-degree. Vertical noise is in metres. -->
         <position_sensing>
           <horizontal><noise type="gaussian"><mean>0.0</mean><stddev>${gps_noise_m / 111320.0}</stddev></noise></horizontal>
-          <vertical><noise type="gaussian"><mean>0.0</mean><stddev>0.5</stddev></noise></vertical>
+          <vertical><noise type="gaussian"><mean>0.0</mean><stddev>0.02</stddev></noise></vertical>
         </position_sensing>
       </navsat>
